Commit message: heron_description: solved location error of painting tanks mesh

File: heron_description/urdf/structures/painting_tools.urdf.xacro (robot description, xacro)
@@ -20,5 +20,5 @@
                 </material>
                 <geometry>
-                    <mesh filename="package://heron_bringup/meshes/structures/painting_tanks.stl"/>
+                    <mesh filename="package://heron_description/meshes/structures/painting_tanks.stl"/>
                 </geometry>
             </visual>
@@ -26,5 +26,5 @@
             <origin rpy="0 0 0" xyz="0 0 0"/>
             <geometry>
-                <mesh filename="package://heron_bringup/meshes/structures/painting_tanks.stl"/>
+                <mesh filename="package://heron_description/meshes/structures/painting_tanks.stl"/>
             </geometry>
             </collision>
