Commit message: heron_description: changed location of painting tool set, corrected parent link of the arm

File: heron_description/robots/heron.urdf.xacro (robot description, xacro)
@@ -35,7 +35,7 @@
     <!-- Imports robot -->
     <!--xacro:include filename="$(find heron)/urdf/robots/rbvogui_xl.urdf.xacro" /-->
-    <xacro:include filename="$(find heron_bringup)/urdf/robots/rbvogui_xl.urdf.xacro" />
+    <xacro:include filename="$(find heron_description)/robots/rbvogui_xl.urdf.xacro" />
     <!-- Imports painting tools -->
-    <xacro:include filename="$(find heron_bringup)/urdf/robots/painting_tools.urdf.xacro" />
+    <xacro:include filename="$(find heron_description)/urdf/structures/painting_tools.urdf.xacro" />
     <!-- Declares specific elements depending on the use case -->
     <xacro:macro name="heron" params="prefix use_case">

File: heron_description/robots/rbvogui_xl.urdf.xacro (robot description, xacro)
@@ -101,5 +101,5 @@
         <joint name="${prefix}arm_base_joint" type="fixed">
             <origin xyz="0 0 0.508" rpy="0 0 ${PI/4}"/>
-            <parent link="${prefix}ewellix_lift_2_link" />
+            <parent link="${prefix}ewellix_lift_top_link" />
             <child link="${prefix}arm_base_link" />
         </joint>

File: heron_description/urdf/structures/painting_tools.urdf.xacro (robot description, xacro)
@@ -20,5 +20,5 @@
                 </material>
                 <geometry>
-                    <mesh filename="package://heron_bringup/meshes/painting_tanks.stl"/>
+                    <mesh filename="package://heron_bringup/meshes/structures/painting_tanks.stl"/>
                 </geometry>
             </visual>
@@ -26,5 +26,5 @@
             <origin rpy="0 0 0" xyz="0 0 0"/>
             <geometry>
-                <mesh filename="package://heron_bringup/meshes/painting_tanks.stl"/>
+                <mesh filename="package://heron_bringup/meshes/structures/painting_tanks.stl"/>
             </geometry>
             </collision>

Commit message: heron_description: Added cones tool set

File: heron_description/robots/heron.urdf.xacro (robot description, xacro)
@@ -38,4 +38,6 @@
     <!-- Imports painting tools -->
     <xacro:include filename="$(find heron_description)/urdf/structures/painting_tools.urdf.xacro" />
+    <!-- Imports cones tools -->
+    <xacro:include filename="$(find heron_description)/urdf/structures/cones_tools.urdf.xacro" />
     <!-- Declares specific elements depending on the use case -->
     <xacro:macro name="heron" params="prefix use_case">
@@ -48,6 +50,5 @@
       <!--Road marks use case: Cones box + 3FG15 gripper -->
       <xacro:if value="${use_case == 'cones'}">
-        <xacro:cones_tools prefix="${prefix}painting_" parent="${prefix}chassis_link">
-            <origin xyz="-0.0475 0 0.287" rpy="1.57 0 -1.57"/>
+        <xacro:cones_tools prefix="${prefix}cones_">
         </xacro:cones_tools>
       </xacro:if>
