Commit message: changed collisions of logos and charging contacts

File: heron_description/urdf/bases/rbvogui_xl_base.urdf.xacro (robot description, xacro)
@@ -122,4 +122,10 @@
         </material>
       </visual>
+      <collision>
+        <origin xyz="0 0 0" rpy="0 0 0" />
+        <geometry>
+          <mesh filename="package://rbvogui_description/meshes/bases/rbvogui_contactors.stl" />
+        </geometry>
+      </collision>
     </link>
     <!-- Logos -->
@@ -133,18 +139,17 @@
       <visual>
         <origin xyz="0 0 -0.06" rpy="0 0 0" />
-        <xacro:if value="${hq}">
-          <geometry>
-            <mesh filename="package://rbvogui_description/meshes/bases/rbvogui_logos.stl" scale="1.24 1.24 1"/>
-          </geometry>
-        </xacro:if>
-        <xacro:unless value="${hq}">
-          <geometry>
-            <mesh filename="package://rbvogui_description/meshes/bases/rbvogui_logos.dae" scale="1.3 1.3 1"/>
-          </geometry>
-        </xacro:unless>
+        <geometry>
+          <mesh filename="package://rbvogui_description/meshes/bases/rbvogui_logos.stl" scale="1.24 1.24 1"/>
+        </geometry>
         <material name="lightred">
           <color rgba="0.9 0.2 0.2 1"/>
         </material>
       </visual>
+      <collision>
+        <origin xyz="0 0 -0.06" rpy="0 0 0" />
+        <geometry>
+          <mesh filename="package://rbvogui_description/meshes/bases/rbvogui_logos.stl" />
+        </geometry>
+      </collision>
     </link>
     <joint name="${prefix}leds_joint" type="fixed">
@@ -163,4 +168,10 @@
         </material>
       </visual>
+      <collision>
+        <origin xyz="0 0 0" rpy="0 0 0.0" />
+        <geometry>
+            <mesh filename="package://rbvogui_description/meshes/bases/rbvogui_xl_leds.stl" />
+        </geometry>
+      </collision>
     </link>
     <xacro:gazebo_color_base_link prefix="${prefix}"/>
